Commit message: Update rover.urdf
Fix rover scale for better RViz2 visualization

File: rover.urdf (robot description, URDF)
Before this commit: robot rover, 9 links, 8 joints
Links:
- link back_left_wheel: geometry collision mesh filename=back_left_wheel.stl scale=0.1 0.1 0.1; visual mesh filename=back_left_wheel.stl scale=0.1 0.1 0.1
- link back_right_wheel: geometry collision mesh filename=back_right_wheel.stl scale=0.1 0.1 0.1; visual mesh filename=back_right_wheel.stl scale=0.1 0.1 0.1
- link base_link: geometry collision mesh filename=Base.stl scale=0.1 0.1 0.1; visual mesh filename=Base.stl scale=0.1 0.1 0.1
- link battery: geometry visual mesh filename=battery.stl scale=0.1 0.1 0.1
- link camera: geometry visual mesh filename=camera.stl scale=0.1 0.1 0.1
- link front_left_wheel: geometry collision mesh filename=front_left_wheel.stl scale=0.1 0.1 0.1; visual mesh filename=front_left_wheel.stl scale=0.1 0.1 0.1
- link front_right_wheel: geometry collision mesh filename=front_right_wheel.stl scale=0.1 0.1 0.1; visual mesh filename=front_right_wheel.stl scale=0.1 0.1 0.1
- link lidar: geometry visual mesh filename=lidar.stl scale=0.1 0.1 0.1
- link motherboard: geometry visual mesh filename=motherboard.stl scale=0.1 0.1 0.1
